File: PCB/pico_plus.kicad_sch (KiCad schematic)
At the start: 36 parts, among them J1 USB_C_Receptacle_USB2.0_16P, SW1 SW_Push, SW2 SW_Push, U1 RP2350_60QFN, U2 TLV1117-33, U3 W25Q128JVS, U4 AT25M02, Y1 ABM8-272-T3

Commit message: Some work on schematic
Parts:
- removed U4: AT25M02, symbol Memory_EEPROM:AT25xxx
Changed lines of the file:
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@@
-	)
-	(symbol
-		(lib_id "Memory_EEPROM:AT25xxx")
-		(at 85.09 175.26 0)
-		(unit 1)
-		(exclude_from_sim no)
-		(in_bom yes)
-		(on_board yes)
-		(dnp no)
-		(fields_autoplaced yes)
-		(property "Reference" "U4"
-			(at 87.2333 165.1 0)
-			(effects
-				(font
-					(size 1.27 1.27)
-				)
-				(justify left)
-			)
-		)
-		(property "Value" "AT25M02"
-			(at 87.2333 167.64 0)
-			(effects
-				(font
-					(size 1.27 1.27)
-				)
-				(justify left)
-			)
-		)
-		(property "Footprint" ""
-			(at 85.09 175.26 0)
-			(effects
-				(font
-					(size 1.27 1.27)
-				)
-				(hide yes)
-			)
-		)
-		(property "Datasheet" "http://ww1.microchip.com/downloads/en/DeviceDoc/Atmel-8707-SEEPROM-AT25010B-020B-040B-Datasheet.pdf"
-			(at 85.09 175.26 0)
-			(effects
-				(font
-					(size 1.27 1.27)
-				)
-				(hide yes)
-			)
-		)
-		(property "Description" "Microchip SPI Serial EEPROM, DIP-8/SOIC-8/TSSOP-8"
-			(at 85.09 175.26 0)
-			(effects
-				(font
-					(size 1.27 1.27)
-				)
-				(hide yes)
-			)
-		)
-		(pin "7"
-		)
-		(pin "8"
-		)
-		(pin "5"
-		)
-		(pin "1"
-		)
-		(pin "4"
-		)
-		(pin "3"
-		)
-		(pin "6"
-		)
-		(pin "2"
-		)
-		(instances
-			(project ""
-				(path "/178505cd-8ab7-4104-a7aa-1c5f6363b7ad"
-					(reference "U4")
-					(unit 1)
-				)
-			)
-		)
 	)
 	(symbol

Commit message: a lot of work
Parts:
- added X1: ~, symbol Pico:Pico
Connections:
- net +3.3V is gone; now on net +3V3: TP2.1, U2.2 (VO)
- net +3V3: now also X1.36 (3V3_OUT), X1.39 (VSYS)
- net GND: now also X1.13 (GND), X1.18 (GND), X1.23 (GND), X1.28 (GND), X1.3 (GND), X1.33 (GND), X1.38 (GND), X1.8 (GND), X1.GND
- net GP0: now also X1.1 (GP0)
- net GP1: now also X1.2 (GP1)
- net GP10: now also X1.14 (GP10)
- net GP11: now also X1.15 (GP11)
- net GP12: now also X1.16 (GP12)
- net GP13: now also X1.17 (GP13)
- net GP15: now also X1.19 (GP14)
- net GP16: now also X1.20 (GP15), X1.22 (GP17)
- net GP17: now also X1.21 (GP16)
- net GP18: now also X1.27 (GP21)
- net GP19: now also X1.26 (GP20)
- net GP2: now also X1.4 (GP2)
- net GP20: now also X1.25 (GP19)
- net GP21: now also X1.24 (GP18)
- net GP22: now also X1.29 (GP22)
- net GP3: now also X1.5 (GP3)
- net GP4: now also X1.6 (GP4)
- net GP5: now also X1.7 (GP5)
- net GP6: now also X1.9 (GP6)
- net GP7: now also X1.10 (GP7)
- net GP8: now also X1.11 (GP8)
- net GP9: now also X1.12 (GP9)
- net RUN: now also X1.30 (RUN)
- net +5V renamed VBUS
- net VBUS: now also X1.40 (VBUS)
- net GP26 renamed GP26_ADC0
- net GP26_ADC0: now also X1.32 (GP27)
- net GP27 renamed GP27_ADC1
- net GP27_ADC1: now also X1.31 (GP26)
- net GP28 renamed GP28_ADC2
- net GP28_ADC2: now also X1.34 (GP28)
- net GP29 renamed GP29_ADC3
- net GP29_ADC3: now also X1.37 (3V3_EN)

Commit message: finish schematic
Parts:
- removed R9: DNF, Resistor_SMD:R_0402_1005Metric, symbol Device:R
- added C19: 4.7uF, Capacitor_SMD:C_0402_1005Metric, symbol Device:C
- added C20, C21: 4.7u, Capacitor_SMD:C_0402_1005Metric, symbol Device:C
- added C22: 4.7u, Resistor_SMD:R_0805_2012Metric, symbol Device:C
- added C23: 100n, Capacitor_SMD:C_0402_1005Metric, symbol Device:C
- added D1: B5819W SL, Diode_SMD:D_SOD-123, symbol Device:D_Schottky
- added D2: LED Green, LED_SMD:LED_0805_2012Metric, symbol Device:LED
- added JP1: SolderJumper_2_Bridged, Jumper:SolderJumper-2_P1.3mm_Bridged2Bar_RoundedPad1.0x1.5mm, symbol Jumper:SolderJumper_2_Bridged
- added L1: 3.3u, Components:AOTA-B201610S3R3-101-T, symbol Device:L
- added R11: 200, Resistor_SMD:R_0402_1005Metric, symbol Device:R
- added R12: 1, Resistor_SMD:R_0603_1608Metric, symbol Device:R
- added R13: 470, Resistor_SMD:R_0402_1005Metric, symbol Device:R
- added R14: 33, Resistor_SMD:R_0402_1005Metric, symbol Device:R
- added R15: 10k, Resistor_SMD:R_0402_1005Metric, symbol Device:R
- added TP6: LED_TP, TestPoint:TestPoint_Pad_D1.5mm, symbol Connector:TestPoint
- added U4: APS6404L-3SQR-ZR, Components:PSON50P200X300X50-9N, symbol APS6404L-3SQR-ZR:APS6404L-3SQR-ZR
- added U5: AT24CM02-SSHM-T, Package_SO:SOIC-8_3.9x4.9mm_P1.27mm, symbol AT24CM02_SSHM_T:AT24CM02-SSHM-T
- J1: footprint (none) -> Connector_USB:USB_C_Receptacle_GCT_USB4105-xx-A_16P_TopMnt_Horizontal
- R1, R2, R3, R4, R5: footprint (none) -> Resistor_SMD:R_0402_1005Metric
- R10: value 0 -> 10k
- R8: value 10k / DNF -> 10k
- U2: footprint (none) -> Package_TO_SOT_SMD:SOT-223
- X1: footprint (none) -> Library:Pico_Castellated_Holes
- Y1: footprint (none) -> RP2350_60QFN_minimal:Crystal_SMD_HC49-US
Connections:
- net +1V1: now also C21.1, L1.2
- net +3V3: now also R10.2, U1.49 (VREG_VIN), C19.1, C22.1, C23.1, R11.1, R12.2, R14.2, R15.2, U4.8 (VDD), U5.8 (VCC); no longer X1.39 (VSYS)
- net GND: now also U1.47 (VREG_PGND), C19.2, C20.2, C21.2, C22.2, C23.2, D2.1 (K), U4.4 (VSS), U4.9 (EXP), U5.3 (A2), U5.4 (GND), U5.7 (WP)
- net GP0: now also JP1.1 (A)
- net GP14: now also X1.19 (GP14)
- net GP15: now also X1.20 (GP15); no longer X1.19 (GP14)
- net GP16: now also X1.21 (GP16); no longer X1.20 (GP15), X1.22 (GP17)
- net GP17: now also X1.22 (GP17); no longer X1.21 (GP16)
- net GP18: now also X1.24 (GP18); no longer X1.27 (GP21)
- net GP19: now also X1.25 (GP19); no longer X1.26 (GP20)
- net GP20: now also X1.26 (GP20); no longer X1.25 (GP19)
- net GP21: now also X1.27 (GP21); no longer X1.24 (GP18)
- net GP23: now also U5.6 (SCL)
- net GP24: now also U5.5 (SDA)
- net GP25: now also R13.1
- net GP26_ADC0: now also X1.31 (GP26); no longer X1.32 (GP27)
- net GP27_ADC1: now also X1.32 (GP27); no longer X1.31 (GP26)
- net QSPI_SD0: now also U4.5 (SI/SIO(0))
- net QSPI_SD1: now also U4.2 (SO/SIO(1))
- net QSPI_SD2: now also U4.3 (SIO(2))
- net QSPI_SD3: now also U4.7 (SIO(3))
- net QSPI_SS: no longer R10.2
- net VBUS: now also D1.2 (A); no longer U2.3 (VI)
- net ADC_VREF: now reaches X1.35 (ADC_VREF)
- net ADC_VREF: now also R11.2, R12.1
- net VREG_AVDD: now reaches U1.46 (VREG_AVDD)
- net VREG_AVDD: now also C20.1, R14.1
- net VREG_FB: now reaches U1.50 (VREG_FB)
- net VREG_FB: now also L1.1
- net ~{USB_BOOT} renamed USB_BOOT
- new net: D2.2 (A), R13.2, TP6.1
- new net RAM_CE: JP1.2 (B), R15.1, U4.1 (~{CE})
- new net RAM_SCLK: U4.6 (SCLK)
- new net VSYS: D1.1 (K), U2.3 (VI), X1.39 (VSYS)
Other:
- note added: "GPIO0 is a QMI CS1n pin. Because we are using the RP2350A variant, there's only 3 of these gpio pins. I've determined that GPIO0 is the most "out of the way""
- note added: "I2C EEPROM"
- note added: "PSRAM Chip (APS6505L - 8MB)"
- note added: "Quartz Clock"
- note added: "pull chip select to 3v3"
- moved on the sheet: C12, C13, C14, C15, C16, C17, C18, C2, C3, C4, R10, R5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

Commit message: work on pcb
Parts:
- TP1, TP2, TP3, TP4, TP5, TP6: footprint TestPoint:TestPoint_Pad_D1.5mm -> TestPoint:TestPoint_Pad_D1.0mm
- Y1: footprint RP2350_60QFN_minimal:Crystal_SMD_HC49-US -> RP2350_60QFN_minimal:XTAL_ABM8-272-T3
Connections:
- net SWCLK: now also X1.SWCLK
- net SWD: now also X1.SWDIO
Changed lines of the file:
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@@
 	(wire
 		(pts
+			(xy 340.36 184.15) (xy 340.36 175.26)
+		)
+		(stroke
+			(width 0)
+			(type default)
+		)
+	)
+	(wire
+		(pts
 			(xy 173.99 60.96) (xy 185.42 60.96)
 		)
@@
 	(wire
 		(pts
+			(xy 337.82 186.69) (xy 337.82 175.26)
+		)
+		(stroke
+			(width 0)
+			(type default)
+		)
+	)
+	(wire
+		(pts
 			(xy 229.87 71.12) (xy 233.68 71.12)
 		)
@@
 	(wire
 		(pts
+			(xy 335.28 184.15) (xy 335.28 175.26)
+		)
+		(stroke
+			(width 0)
+			(type default)
+		)
+	)
+	(wire
+		(pts
 			(xy 364.49 135.89) (xy 351.79 135.89)
 		)
@@
 		)
 	)
+	(label "SWCLK"
+		(at 335.28 184.15 90)
+		(effects
+			(font
+				(size 1.27 1.27)
+			)
+			(justify left bottom)
+		)
+	)
 	(label "GP1"
 		(at 257.81 100.33 180)
@@
 		)
 	)
+	(label "SWD"
+		(at 340.36 184.15 90)
+		(effects
+			(font
+				(size 1.27 1.27)
+			)
+			(justify left bottom)
+		)
+	)
 	(label "GP25"
 		(at 257.81 161.29 180)
@@
 	(symbol
 		(lib_id "power:GND")
-		(at 337.82 175.26 0)
+		(at 337.82 186.69 0)
 		(mirror y)
 		(unit 1)
@@
 		(dnp no)
 		(property "Reference" "#PWR037"
-			(at 337.82 181.61 0)
+			(at 337.82 193.04 0)
 			(effects
 				(font
@@
 		)
 		(property "Value" "GND"
-			(at 337.693 179.6542 0)
+			(at 337.693 191.0842 0)
 			(effects
 				(font
@@
 		)
 		(property "Footprint" ""
-			(at 337.82 175.26 0)
+			(at 337.82 186.69 0)
 			(effects
 				(font
@@
 		)
 		(property "Datasheet" ""
-			(at 337.82 175.26 0)
+			(at 337.82 186.69 0)
 			(effects
 				(font
@@
 		)
 		(property "Description" ""
-			(at 337.82 175.26 0)
+			(at 337.82 186.69 0)
 			(effects
 				(font
@@
 			)
 		)
-		(property "Footprint" "TestPoint:TestPoint_Pad_D1.5mm"
+		(property "Footprint" "TestPoint:TestPoint_Pad_D1.0mm"
 			(at 125.73 31.75 0)
 			(effects
@@
 		(pin "23"
 		)
+		(pin "SWDIO"
+		)
+		(pin "SWCLK"
+		)
 		(instances
 			(project ""
@@
 			)
 		)
-		(property "Footprint" "TestPoint:TestPoint_Pad_D1.5mm"
+		(property "Footprint" "TestPoint:TestPoint_Pad_D1.0mm"
 			(at 30.48 50.8 0)
 			(effects
@@
 			)
 		)
-		(property "Footprint" "TestPoint:TestPoint_Pad_D1.5mm"
+		(property "Footprint" "TestPoint:TestPoint_Pad_D1.0mm"
 			(at 72.39 31.75 0)
 			(effects
@@
 			)
 		)
-		(property "Footprint" "TestPoint:TestPoint_Pad_D1.5mm"
+		(property "Footprint" "TestPoint:TestPoint_Pad_D1.0mm"
 			(at 17.78 50.8 0)
 			(effects
@@
 			)
 		)
-		(property "Footprint" "RP2350_60QFN_minimal:Crystal_SMD_HC49-US"
+		(property "Footprint" "RP2350_60QFN_minimal:XTAL_ABM8-272-T3"
 			(at 71.12 210.82 0)
 			(effects
@@
 			)
 		)
-		(property "Footprint" "TestPoint:TestPoint_Pad_D1.5mm"
+		(property "Footprint" "TestPoint:TestPoint_Pad_D1.0mm"
 			(at 353.06 81.28 0)
 			(effects
@@
 			)
 		)
-		(property "Footprint" "TestPoint:TestPoint_Pad_D1.5mm"
+		(property "Footprint" "TestPoint:TestPoint_Pad_D1.0mm"
 			(at 29.21 63.5 0)
 			(effects

Commit message: temp
Parts:
- removed R10: 10k, Resistor_SMD:R_0402_1005Metric, symbol Device:R
- removed U3: W25Q128JVS, Package_SO:SOIC-8_5.3x5.3mm_P1.27mm, symbol Memory_Flash:W25Q128JVS
- removed U5: AT24CM02-SSHM-T, Package_SO:SOIC-8_3.9x4.9mm_P1.27mm, symbol AT24CM02_SSHM_T:AT24CM02-SSHM-T
- added D3: WS2812B, LED_SMD:LED_WS2812B_PLCC4_5.0x5.0mm_P3.2mm, symbol LED:WS2812B
- added J3: Conn_01x01, Connector_PinHeader_2.54mm:PinHeader_1x01_P2.54mm_Vertical, symbol Connector_Generic:Conn_01x01
- added SW3: SW_Push, Components:SW-SMD_L3.9-W3.0-P4.45, symbol Switch:SW_Push
- added U3: W25Q128JVP, Package_SON:WSON-8-1EP_6x5mm_P1.27mm_EP3.4x4.3mm, symbol Memory_Flash:W25Q128JVP
- C10, C11, C12, C13, C14, C15, C16, C17, C18, C19, C2, C20, C21, C23, C3, C4, C8: footprint Capacitor_SMD:C_0402_1005Metric -> Capacitor_SMD:C_0201_0603Metric
- C22: footprint Resistor_SMD:R_0805_2012Metric -> Capacitor_SMD:C_0201_0603Metric
- R1, R11, R13, R14, R15, R2, R3, R4, R5, R6, R7, R8: footprint Resistor_SMD:R_0402_1005Metric -> Resistor_SMD:R_0201_0603Metric
- R12: footprint Resistor_SMD:R_0603_1608Metric -> Resistor_SMD:R_0201_0603Metric
- SW1, SW2: footprint Button_Switch_SMD:SW_Push_1P1T_NO_Vertical_Wuerth_434133025816 -> Components:SW-SMD_L3.9-W3.0-P4.45
- U2: footprint Package_TO_SOT_SMD:SOT-223 -> Package_TO_SOT_SMD:SOT-223-3_TabPin2
Connections:
- net +3V3: now also U3.8 (VCC)
- net GND: now also D3.3 (VSS), SW3.2, U3.4 (GND), U3.9 (EP)
- net GP23: now also D3.4 (DIN)
- net GP24: now also SW3.1
- net QSPI_SCLK: now also U3.6 (CLK)
- net QSPI_SD0: now also U3.5 (DI/IO_{0})
- net QSPI_SD1: now also U3.2 (DO/IO_{1})
- net QSPI_SD2: now also U3.3 (~{WP}/IO_{2})
- net QSPI_SD3: now also U3.7 (~{HOLD}/~{RESET}/IO_{3})
- net QSPI_SS: now also U3.1 (~{CS})
- net VSYS: now also D3.1 (VDD)
- new net: D3.2 (DOUT), J3.1 (Pin_1)
Other:
- note removed: "I2C EEPROM"

Commit message: finish routing
Parts:
- removed J3: Conn_01x01, Connector_PinHeader_2.54mm:PinHeader_1x01_P2.54mm_Vertical, symbol Connector_Generic:Conn_01x01
- removed JP1: SolderJumper_2_Bridged, Jumper:SolderJumper-2_P1.3mm_Bridged2Bar_RoundedPad1.0x1.5mm, symbol Jumper:SolderJumper_2_Bridged
- removed U2: TLV1117-33, Package_TO_SOT_SMD:SOT-223-3_TabPin2, symbol Regulator_Linear:TLV1117-33
- added R16: 10k, Resistor_SMD:R_0201_0603Metric, symbol Device:R
- added TP7: LEDOUT, TestPoint:TestPoint_Pad_D1.0mm, symbol Connector:TestPoint
- added U2: TPS7A20xxxDQN, Package_SON:Texas_X2SON-4_1x1mm_P0.65mm, symbol Regulator_Linear:TPS7A20xxxDQN
- C21, C22: footprint Capacitor_SMD:C_0201_0603Metric -> RP2350_60QFN_minimal:C_0402_1005Metric_small_pads
- L1: footprint Components:AOTA-B201610S3R3-101-T -> RP2350_60QFN_minimal:L_pol_2016
Connections:
- net RAM_CE is gone; now on net GP0: R15.1, U4.1 (~{CE})
- net VREG_FB is gone; now on net +1V1: L1.1, U1.50 (VREG_FB)
- net +1V1: no longer L1.2
- net +3V3: now also U2.1 (OUT)
- net GND: now also U2.2 (GND), U2.5 (Pad)
- net GP29_ADC3: no longer X1.37 (3V3_EN)
- net VREG_LX: now also L1.2
- net VSYS: now also R16.1, U2.4 (IN)
- net at D3.2 (DOUT): now also TP7.1
- new net 3V3_EN: R16.2, U2.3 (EN), X1.37 (3V3_EN)
Other:
- moved on the sheet: L1

Commit message: finish pcb
Parts:
- removed TP1: VBUS_TP, TestPoint:TestPoint_Pad_D1.0mm, symbol Connector:TestPoint
- removed TP3: GND_TP, TestPoint:TestPoint_Pad_D1.0mm, symbol Connector:TestPoint
- removed TP4: DP_TP, TestPoint:TestPoint_Pad_D1.0mm, symbol Connector:TestPoint
- removed TP5: DM_TP, TestPoint:TestPoint_Pad_D1.0mm, symbol Connector:TestPoint
- added JP1: SolderJumper_2_Bridged, Jumper:SolderJumper-2_P1.3mm_Bridged2Bar_RoundedPad1.0x1.5mm, symbol Jumper:SolderJumper_2_Bridged
Connections:
- net GP0: now also JP1.1 (A); no longer R15.1, U4.1 (~{CE})
- new net RAM_CE: JP1.2 (B), R15.1, U4.1 (~{CE})

Commit message: schematic fix
Other:
- note added: "PSRAM Chip (APS6404L - 8MB)"
- note removed: "PSRAM Chip (APS6505L - 8MB)"
Changed lines of the file:
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@@
 		)
 	)
-	(text "PSRAM Chip\n(APS6505L - 8MB)"
+	(text "PSRAM Chip\n(APS6404L - 8MB)"
 		(exclude_from_sim no)
 		(at 77.216 133.858 0)
