File: PCB/pico_plus.kicad_pcb (KiCad board)
At the start: 2 copper layers, 21 x 51 mm, 1 part

Commit message: finish schematic
Parts:
- removed REF**: Pico_Castellated_Holes, Library:Pico_Castellated_Holes
- added C10: 4.7u, Capacitor_SMD:C_0402_1005Metric, F.Cu at (150.1, 85.3)
- added C11: 100n, Capacitor_SMD:C_0402_1005Metric, F.Cu at (150.1, 87.3)
- added C12: 100n, Capacitor_SMD:C_0402_1005Metric, F.Cu at (150.1, 89.2)
- added C13: 100n, Capacitor_SMD:C_0402_1005Metric, F.Cu at (153.0, 77.4)
- added C14: 100n, Capacitor_SMD:C_0402_1005Metric, F.Cu at (153.0, 79.4)
- added C15: 100n, Capacitor_SMD:C_0402_1005Metric, F.Cu at (153.0, 81.3)
- added C16: 100n, Capacitor_SMD:C_0402_1005Metric, F.Cu at (153.0, 83.3)
- added C17: 100n, Capacitor_SMD:C_0402_1005Metric, F.Cu at (153.0, 85.3)
- added C18: 100n, Capacitor_SMD:C_0402_1005Metric, F.Cu at (153.0, 87.3)
- added C19: 4.7uF, Capacitor_SMD:C_0402_1005Metric, F.Cu at (153.0, 89.2)
- added C2: 100n, Capacitor_SMD:C_0402_1005Metric, F.Cu at (150.1, 77.4)
- added C20: 4.7u, Capacitor_SMD:C_0402_1005Metric, F.Cu at (155.8, 77.4)
- added C21: 4.7u, Capacitor_SMD:C_0402_1005Metric, F.Cu at (155.8, 79.4)
- added C22: 4.7u, Resistor_SMD:R_0805_2012Metric, F.Cu at (155.8, 81.3)
- added C23: 100n, Capacitor_SMD:C_0402_1005Metric, F.Cu at (155.8, 83.3)
- added C3: 15p, Capacitor_SMD:C_0402_1005Metric, F.Cu at (150.1, 79.4)
- added C4: 15p, Capacitor_SMD:C_0402_1005Metric, F.Cu at (150.1, 81.3)
- added C8: 100n, Capacitor_SMD:C_0402_1005Metric, F.Cu at (150.1, 83.3)
- added D1: B5819W SL, Diode_SMD:D_SOD-123, F.Cu at (162.2, 116.9)
- added D2: LED Green, LED_SMD:LED_0805_2012Metric, F.Cu at (159.5, 87.9)
- added J1: USB_C_Receptacle_USB2.0_16P, Connector_USB:USB_C_Receptacle_GCT_USB4105-xx-A_16P_TopMnt_Horizontal, F.Cu at (119.0, 71.6)
- added JP1: SolderJumper_2_Bridged, Jumper:SolderJumper-2_P1.3mm_Bridged2Bar_RoundedPad1.0x1.5mm, F.Cu at (166.4, 92.0)
- added L1: 3.3u, Components:AOTA-B201610S3R3-101-T, F.Cu at (163.7, 88.3)
- added R1: 5.1k, Resistor_SMD:R_0402_1005Metric, F.Cu at (150.7, 65.1)
- added R10: 10k, Resistor_SMD:R_0402_1005Metric, F.Cu at (154.7, 72.7)
- added R11: 200, Resistor_SMD:R_0402_1005Metric, F.Cu at (154.7, 75.2)
- added R12: 1, Resistor_SMD:R_0603_1608Metric, F.Cu at (158.7, 65.1)
- added R13: 470, Resistor_SMD:R_0402_1005Metric, F.Cu at (158.7, 67.6)
- added R14: 33, Resistor_SMD:R_0402_1005Metric, F.Cu at (158.7, 70.2)
- added R15: 10k, Resistor_SMD:R_0402_1005Metric, F.Cu at (158.7, 72.7)
- added R2: 5.1k, Resistor_SMD:R_0402_1005Metric, F.Cu at (150.7, 67.6)
- added R3: 27, Resistor_SMD:R_0402_1005Metric, F.Cu at (150.7, 70.2)
- added R4: 27, Resistor_SMD:R_0402_1005Metric, F.Cu at (150.7, 72.7)
- added R5: 1k, Resistor_SMD:R_0402_1005Metric, F.Cu at (150.7, 75.2)
- added R6: 1k, Resistor_SMD:R_0402_1005Metric, F.Cu at (154.7, 65.1)
- added R7: 1k, Resistor_SMD:R_0402_1005Metric, F.Cu at (154.7, 67.6)
- added R8: 10k, Resistor_SMD:R_0402_1005Metric, F.Cu at (154.7, 70.2)
- added SW1: SW_Push, Button_Switch_SMD:SW_Push_1P1T_NO_Vertical_Wuerth_434133025816, F.Cu at (162.7, 108.1)
- added SW2: SW_Push, Button_Switch_SMD:SW_Push_1P1T_NO_Vertical_Wuerth_434133025816, F.Cu at (162.7, 112.9)
- added TP1: VBUS_TP, TestPoint:TestPoint_Pad_D1.5mm, F.Cu at (150.4, 107.5)
- added TP2: 3V3_TP, TestPoint:TestPoint_Pad_D1.5mm, F.Cu at (150.4, 111.1)
- added TP3: GND_TP, TestPoint:TestPoint_Pad_D1.5mm, F.Cu at (154.0, 107.5)
- added TP4: DP_TP, TestPoint:TestPoint_Pad_D1.5mm, F.Cu at (154.0, 111.1)
- added TP5: DM_TP, TestPoint:TestPoint_Pad_D1.5mm, F.Cu at (157.5, 107.5)
- added TP6: LED_TP, TestPoint:TestPoint_Pad_D1.5mm, F.Cu at (157.5, 111.1)
- added U1: RP2350_60QFN, RP2350_60QFN_minimal:RP2350-QFN-60-1EP_7x7_P0.4mm_EP3.4x3.4mm_ThermalVias, F.Cu at (141.8, 87.2)
- added U2: TLV1117-33, Package_TO_SOT_SMD:SOT-223, F.Cu at (162.9, 100.7)
- added U3: W25Q128JVS, Package_SO:SOIC-8_5.3x5.3mm_P1.27mm, F.Cu at (153.8, 116.3)
- added U4: APS6404L-3SQR-ZR, Components:PSON50P200X300X50-9N, F.Cu at (163.0, 73.1)
- added U5: AT24CM02-SSHM-T, Package_SO:SOIC-8_3.9x4.9mm_P1.27mm, F.Cu at (164.9, 67.2)
- added X1: ~, Library:Pico_Castellated_Holes, F.Cu at (118.8, 63.1)
- added Y1: ABM8-272-T3, RP2350_60QFN_minimal:Crystal_SMD_HC49-US, F.Cu at (156.5, 93.3)

Commit message: work on pcb
Parts:
- TP1, TP2, TP3, TP4, TP5, TP6: footprint TestPoint:TestPoint_Pad_D1.5mm -> TestPoint:TestPoint_Pad_D1.0mm
- Y1: footprint RP2350_60QFN_minimal:Crystal_SMD_HC49-US -> RP2350_60QFN_minimal:XTAL_ABM8-272-T3
- moved JP1 53.3 mm to (114.0, 82.3), turned to 90 degrees
- moved TP4 49.0 mm to (117.9, 77.9)
- moved R5 41.1 mm to (119.2, 101.6), turned to -90 degrees
- moved C3 39.8 mm to (117.4, 102.1), turned to 180 degrees
- moved Y1 39.1 mm to (119.0, 104.3), turned to 90 degrees
- moved R2 37.9 mm to (113.1, 72.4), turned to -90 degrees
- moved C4 36.0 mm to (120.7, 102.1)
- moved R3 35.7 mm to (119.8, 88.0), turned to -90 degrees
- moved R4 35.4 mm to (118.8, 88.0), turned to 90 degrees
- moved C10 34.1 mm to (119.2, 99.6), turned to -90 degrees
- moved U5 29.8 mm to (139.0, 81.9)
- moved R1 26.9 mm to (124.8, 72.4), turned to 90 degrees
- moved U1 23.7 mm to (119.0, 93.4)
Routing:
- net /SWCLK: track 0.00 -> 22.7 mm, vias 0 -> 1
- net /GP1: track 0.00 -> 22.5 mm
- net /SWD: track 0.00 -> 21.1 mm, vias 0 -> 1
- net /D+: track 0.00 -> 16.7 mm
- net /GP3: track 0.00 -> 15.6 mm
- net /D-: track 0.00 -> 14.7 mm, vias 0 -> 2
- net /GP4: track 0.00 -> 14.1 mm
- net /GP5: track 0.00 -> 12.1 mm
- net /XIN: track 0.00 -> 9.36 mm
- net /GP0: track 0.00 -> 9.28 mm
- net /GP6: track 0.00 -> 7.62 mm
- net /GP7: track 0.00 -> 6.33 mm
- net /GP9: track 0.00 -> 6.20 mm
- net Net-(J1-CC1): track 0.00 -> 5.95 mm
- net Net-(J1-CC2): track 0.00 -> 5.61 mm
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- added copper zone on F.Cu, net +1V1
- added copper zone on F.Cu, net +3V3
- added copper zone on B.Cu, net GND
- added copper zone on F.Cu, net GND

Commit message: temp
Parts:
- removed R10: 10k, Resistor_SMD:R_0402_1005Metric
- removed U5: AT24CM02-SSHM-T, Package_SO:SOIC-8_3.9x4.9mm_P1.27mm
- added D3: WS2812B, LED_SMD:LED_WS2812B_PLCC4_5.0x5.0mm_P3.2mm, F.Cu at (119.0, 111.4)
- added J3: Conn_01x01, Connector_PinHeader_2.54mm:PinHeader_1x01_P2.54mm_Vertical, F.Cu at (112.8, 117.2)
- added SW3: SW_Push, Components:SW-SMD_L3.9-W3.0-P4.45, F.Cu at (124.5, 111.2)
- JP1, TP4: moved to B.Cu
- SW1, SW2: footprint Button_Switch_SMD:SW_Push_1P1T_NO_Vertical_Wuerth_434133025816 -> Components:SW-SMD_L3.9-W3.0-P4.45
- U2: footprint Package_TO_SOT_SMD:SOT-223 -> Package_TO_SOT_SMD:SOT-223-3_TabPin2
- U3: value W25Q128JVS -> W25Q128JVP; footprint Package_SO:SOIC-8_5.3x5.3mm_P1.27mm -> Package_SON:WSON-8-1EP_6x5mm_P1.27mm_EP3.4x4.3mm
- moved R6 57.4 mm to (116.5, 108.0)
- moved D1 57.3 mm to (125.5, 73.0), turned to 90 degrees
- moved U3 53.1 mm to (114.8, 80.2), turned to 90 degrees
- moved SW2 49.2 mm to (113.5, 111.5), turned to 90 degrees
- moved U4 47.9 mm to (116.8, 86.0), turned to 90 degrees
- moved U2 45.6 mm to (122.2, 80.0), turned to 180 degrees
- moved TP1 45.5 mm to (125.5, 69.5)
- moved SW1 44.5 mm to (123.8, 86.5), turned to -90 degrees
- moved R8 43.9 mm to (114.1, 86.8), turned to 90 degrees
- moved R7 38.0 mm to (121.0, 85.2)
- moved C18 38.0 mm to (117.0, 99.5), turned to -135 degrees
- moved C14 31.2 mm to (125.2, 93.8)
- moved C11 25.5 mm to (125.2, 92.8)
- moved L1 24.9 mm to (138.9, 86.8)
- moved TP4 23.2 mm to (104.2, 96.6)
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Routing:
- net +3V3: track 1.69 -> 44.6 mm
- net VBUS: track 0.00 -> 25.4 mm, vias 0 -> 2
- net /GP15: track 0.00 -> 23.7 mm
- net /GP14: track 0.00 -> 21.2 mm
- net VSYS: track 0.00 -> 20.5 mm
- net /RUN: track 0.00 -> 19.5 mm, vias 0 -> 2
- net /GP23: track 0.00 -> 18.7 mm, vias 0 -> 2
- net /GP29_ADC3: track 0.00 -> 18.1 mm, vias 0 -> 1
- net /GP2: track 0.00 -> 17.9 mm, vias 0 -> 1
- net /GP24: track 0.00 -> 16.6 mm
- net /GP13: track 0.00 -> 15.7 mm
- net /D-: track 14.7 -> 0.00 mm, vias 2 -> 0
- net /D+: track 16.7 -> 2.44 mm
- net /GP12: track 0.00 -> 13.0 mm
- net +1V1: track 5.18 -> 16.7 mm, vias 2 -> 6
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
Commit message: finish routing
Parts:
- removed J3: Conn_01x01, Connector_PinHeader_2.54mm:PinHeader_1x01_P2.54mm_Vertical
- removed JP1: SolderJumper_2_Bridged, Jumper:SolderJumper-2_P1.3mm_Bridged2Bar_RoundedPad1.0x1.5mm
- added R16: 10k, Resistor_SMD:R_0201_0603Metric, F.Cu at (125.8, 76.0)
- added TP7: LEDOUT, TestPoint:TestPoint_Pad_D1.0mm, F.Cu at (113.8, 106.7)
- C10, C11, C12, C13, C14, C15, C16, C17, C18, C19, C2, C20, C23, C3, C4, C8: footprint Capacitor_SMD:C_0402_1005Metric -> Capacitor_SMD:C_0201_0603Metric
- C21: footprint Capacitor_SMD:C_0402_1005Metric -> RP2350_60QFN_minimal:C_0402_1005Metric_small_pads
- C22: footprint Resistor_SMD:R_0805_2012Metric -> RP2350_60QFN_minimal:C_0402_1005Metric_small_pads
- L1: footprint Components:AOTA-B201610S3R3-101-T -> RP2350_60QFN_minimal:L_pol_2016
- R1, R11, R13, R14, R15, R2, R3, R4, R5, R6, R7, R8: footprint Resistor_SMD:R_0402_1005Metric -> Resistor_SMD:R_0201_0603Metric
- R12: footprint Resistor_SMD:R_0603_1608Metric -> Resistor_SMD:R_0201_0603Metric
- U2: value TLV1117-33 -> TPS7A20xxxDQN; footprint Package_TO_SOT_SMD:SOT-223-3_TabPin2 -> Package_SON:Texas_X2SON-4_1x1mm_P0.65mm
- moved TP2 47.7 mm to (113.8, 80.6)
- moved R15 46.6 mm to (114.5, 87.5), turned to 90 degrees
- moved C16 43.2 mm to (124.2, 115.5)
- moved TP5 42.6 mm to (119.9, 87.5)
- moved R14 42.2 mm to (122.8, 92.5)
- moved TP6 42.2 mm to (125.5, 83.7)
- moved C23 41.8 mm to (114.5, 89.5), turned to -90 degrees
- moved C13 41.0 mm to (114.7, 92.0), turned to 90 degrees
- moved R12 40.4 mm to (122.2, 82.5), turned to 90 degrees
- moved C17 38.8 mm to (114.2, 86.0), turned to 90 degrees
- moved C21 36.9 mm to (121.0, 91.4)
- moved R13 36.7 mm to (125.0, 82.2)
- moved C22 36.6 mm to (121.0, 92.4)
- moved D2 35.7 mm to (124.5, 80.7)
- moved C2 35.6 mm to (114.5, 79.0), turned to 90 degrees
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Connections:
- L1 pad 1: /VREG_FB -> +1V1
- L1 pad 2: +1V1 -> /VREG_LX
- R15 pad 1: /RAM_CE -> /GP0
- U1 pad 50: /VREG_FB -> +1V1
- U2 pad 1: GND -> +3V3
- U2 pad 2: +3V3 -> GND
- U2 pad 3: VSYS -> /3V3_EN
- U4 pad 1: /RAM_CE -> /GP0
- X1 pad 37: /GP29_ADC3 -> /3V3_EN
Routing:
- net +3V3: track 44.6 -> 100.3 mm, vias 0 -> 1
- net GND: track 9.48 -> 53.3 mm, vias 7 -> 49
- net VSYS: track 20.5 -> 63.8 mm, vias 0 -> 1
- net /QSPI_SD3: track 0.00 -> 29.6 mm, vias 0 -> 4
- net /GP0: track 6.47 -> 31.2 mm, vias 1 -> 3
- net /GP16: track 0.00 -> 20.1 mm
- net /GP25: track 0.00 -> 20.0 mm, vias 0 -> 2
- net /GP29_ADC3: track 18.1 -> 0.00 mm, vias 1 -> 0
- net /QSPI_SD0: track 5.71 -> 23.4 mm, vias 0 -> 2
- net /D-: track 0.00 -> 17.6 mm, vias 0 -> 2
- net /GP17: track 0.00 -> 17.4 mm
- net /D+: track 2.44 -> 18.9 mm, vias 0 -> 2
- net /QSPI_SCLK: track 0.00 -> 16.1 mm, vias 0 -> 2
- net /GP18: track 0.00 -> 12.8 mm
- net /GP19: track 0.00 -> 9.84 mm
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- added copper zone on F.Cu, net /VREG_LX

Commit message: finish pcb
Parts:
- removed TP1: VBUS_TP, TestPoint:TestPoint_Pad_D1.0mm
- removed TP3: GND_TP, TestPoint:TestPoint_Pad_D1.0mm
- removed TP4: DP_TP, TestPoint:TestPoint_Pad_D1.0mm
- removed TP5: DM_TP, TestPoint:TestPoint_Pad_D1.0mm
- added JP1: SolderJumper_2_Bridged, Jumper:SolderJumper-2_P1.3mm_Bridged2Bar_RoundedPad1.0x1.5mm, B.Cu at (113.8, 87.5)
- TP6: moved to B.Cu
- moved D2 23.4 mm to (124.2, 104.1), turned to 90 degrees
- moved R13 19.8 mm to (123.9, 102.0)
- moved TP6 19.5 mm to (123.3, 103.0), turned to 180 degrees
- moved D1 7.07 mm to (122.0, 79.1)
- moved C15 2.88 mm to (124.1, 93.4), turned to 0 degrees
- moved C12 1.76 mm to (124.5, 96.9), turned to 0 degrees
- moved R7 1.15 mm to (118.8, 86.0)
- moved C14 0.92 mm to (113.5, 98.2)
- moved SW1 0.87 mm to (122.9, 86.3)
- moved TP7 0.80 mm to (114.4, 106.2)
- moved C16 0.70 mm to (124.2, 116.2), turned to -45 degrees
- moved C17 0.66 mm to (114.2, 85.3)
- moved R15 0.65 mm to (114.5, 86.8)
- moved C8 0.62 mm to (124.9, 95.6)
- moved R11 0.41 mm to (121.0, 82.4)
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Connections:
- R15 pad 1: /GP0 -> /RAM_CE
- U4 pad 1: /GP0 -> /RAM_CE
Routing:
- net +3V3: track 100.3 -> 84.9 mm
- net /GP25: track 20.0 -> 8.59 mm
- net /QSPI_SD3: track 29.6 -> 19.4 mm
- net VSYS: track 63.8 -> 68.0 mm
- net /RAM_CE: track 0.00 -> 3.73 mm, vias 0 -> 1
- net /GP15: track 22.2 -> 20.1 mm
- net /GP13: track 14.1 -> 12.2 mm
- net GND: track 53.3 -> 55.1 mm, vias 49 -> 64
- net +1V1: track 24.7 -> 22.9 mm
- net /GP8: track 9.80 -> 8.20 mm
- net /D+: track 18.9 -> 17.4 mm
- net /D-: track 17.6 -> 16.2 mm
- net /QSPI_SS: track 15.1 -> 13.9 mm
- net /3V3_EN: track 5.14 -> 6.15 mm
- net Net-(D2-A): track 3.22 -> 2.34 mm, vias 0 -> 1
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- added copper zone on F.Cu, net VBUS
Other:
- board text added: "0"
- board text added: "1"
- board text added: "10"
- board text added: "11"
- board text added: "12"
- board text added: "13"
- board text added: "14"
- board text added: "15"
- board text added: "16"
- board text added: "17"
- board text added: "18"
- board text added: "19"
- board text added: "2"
- board text added: "20"
- board text added: "21"
- board text added: "22"
- board text added: "25"
- board text added: "26"
- board text added: "27"
- board text added: "28"
- board text added: "3"
- board text added: "3V3"
- board text added: "4"
- board text added: "5"
- board text added: "6"
- board text added: "7"
- board text added: "8"
- board text added: "9"
- board text added: "A0"
- board text added: "A1"
- board text added: "A2"
- board text added: "ADC"
- board text added: "BOOT"
- board text added: "EN"
- board text added: "GND"
- board text added: "RST"
- board text added: "RUN"
- board text added: "SWC"
- board text added: "SWD"
- board text added: "USR"
- board text added: "VBUS"
- board text added: "VSYS"
- board text added: "x"

Commit message: finish up pcb + bom
Parts:
- removed TP2: 3V3_TP, TestPoint:TestPoint_Pad_D1.0mm
- C10, C19, C20, C3, C4: footprint Capacitor_SMD:C_0201_0603Metric -> Capacitor_SMD:C_0402_1005Metric
- J1: value USB_C_Receptacle_USB2.0_16P -> ~; footprint Connector_USB:USB_C_Receptacle_GCT_USB4105-xx-A_16P_TopMnt_Horizontal -> Components:USB-C-SMD_TYPE-C-6PIN-2MD-073
- R1, R11, R13, R14, R15, R16, R2, R5, R6, R7, R8: footprint Resistor_SMD:R_0201_0603Metric -> Resistor_SMD:R_0402_1005Metric
- R12: footprint Resistor_SMD:R_0201_0603Metric -> Resistor_SMD:R_0603_1608Metric
- U2: value TPS7A20xxxDQN -> TPS7A2033PDBVR; footprint Package_SON:Texas_X2SON-4_1x1mm_P0.65mm -> Components:SOT-23-5_L2.9-W1.6-P0.95-LS2.8-BR
- moved D1 8.44 mm to (113.6, 79.0)
- moved R12 4.04 mm to (125.7, 83.1), turned to 0 degrees
- moved R11 2.78 mm to (123.8, 82.2)
- moved R2 2.51 mm to (113.2, 70.0)
- moved U2 2.30 mm to (122.5, 79.3)
- moved C4 2.23 mm to (121.6, 106.1), turned to -90 degrees
- moved R1 1.59 mm to (113.2, 72.5)
- moved C2 1.45 mm to (115.4, 77.8), turned to 180 degrees
- moved J1 1.42 mm to (119.0, 73.0)
- moved C20 1.06 mm to (123.2, 90.5), turned to 90 degrees
- moved C23 1.06 mm to (113.5, 89.3)
- moved C19 0.95 mm to (121.9, 82.0), turned to 180 degrees
- moved R16 0.94 mm to (124.9, 75.8), turned to 0 degrees
- moved R15 0.81 mm to (114.3, 87.6)
- moved SW1 0.69 mm to (122.4, 85.8)
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Connections:
- R1 pad 1: Net-(J1-CC1) -> Net-(J1-CC2)
- R2 pad 1: GND -> Net-(J1-CC1)
- R2 pad 2: Net-(J1-CC2) -> GND
- U2 pad 1: +3V3 -> VSYS
- U2 pad 4: VSYS -> unconnected-(U2-NC-Pad4)
- U2 pad 5: GND -> +3V3
Routing:
- net GND: track 55.1 -> 42.9 mm, vias 64 -> 61
- net /3V3_EN: track 6.15 -> 10.3 mm, vias 0 -> 1
- net +3V3: track 84.9 -> 80.7 mm, vias 1 -> 5
- net /ADC_VREF: track 7.40 -> 5.44 mm
- net /GP0: track 31.3 -> 29.4 mm
- net /RUN: track 24.8 -> 26.3 mm
- net Net-(D2-A): track 2.34 -> 3.83 mm
- net VBUS: track 24.0 -> 25.3 mm
- net /D+: track 17.4 -> 16.2 mm
- net /D-: track 16.2 -> 17.2 mm
- net /RAM_CE: track 3.73 -> 3.05 mm
- net /VREG_AVDD: track 2.52 -> 3.19 mm
- net /GP25: track 8.59 -> 8.04 mm
- net VSYS: vias 1 -> 2

Commit message: update bom
Routing:
- net /SWD: track 19.7 -> 19.8 mm, vias 1 -> 2
Other:
- board text added: "1.0"
- board text added: "6/26/2025"
- board text added: "Evan Yu"
- board text added: "Pico+"
